Commit message: fixed teleop

File: ackermann_nav/urdf/ackermann_hokuyo.xacro (robot description, xacro)
@@ -277,3 +277,63 @@
       <joint_properties damping="1.0" friction="1.0" />
     </joint>
+<!-- hokuyo 2d laser scanner -->
+    <joint name="hokuyo_laser_joint" type="fixed">
+        <axis xyz="0 0 1" />
+        <origin xyz="0 0 0.25" rpy="0 0 0"/>
+        <parent link="chassis_link"/>
+        <child link="hokuyo_laser_link"/>
+    </joint>
+    <link name="hokuyo_laser_link">
+        <collision>
+            <origin xyz="0 0 0" rpy="0 0 0"/>
+            <geometry>
+                <cylinder length="0.04" radius="0.045"/>
+            </geometry>
+        </collision>
+        <visual>
+            <origin xyz="0 0 0" rpy="0 0 0"/>
+            <geometry>
+                <cylinder length="0.04" radius="0.045"/>
+            </geometry>
+            <material name="iRobot/LightBlue"/>
+        </visual>
+        <inertial>
+            <mass value="1e-5" />
+            <origin xyz="0 0 0" rpy="0 0 0"/>
+            <inertia ixx="1e-6" ixy="0" ixz="0" iyy="1e-6" iyz="0" izz="1e-6" />
+        </inertial>
+    </link>
+    <gazebo reference="hokuyo_laser_link">
+        <gravity>true</gravity>
+        <sensor type="ray" name="head_hokuyo_sensor">
+            <pose>0 0 0 0 0 0</pose>
+            <visualize>true</visualize>
+            <update_rate>40</update_rate>
+            <ray>
+                <scan>
+                    <horizontal>
+                        <samples>360</samples>
+                        <resolution>1</resolution>
+                        <min_angle>-3.14159</min_angle>
+                        <max_angle>3.14159</max_angle>
+                    </horizontal>
+                </scan>
+                <range>
+                    <min>0.2</min>
+                    <max>40</max>
+                    <resolution>0.025</resolution>
+                </range>
+                <noise>
+                    <type>gaussian</type>
+                    <mean>0.0</mean>
+                    <stddev>0.1</stddev>
+                </noise>
+            </ray>
+            <plugin name="gazebo_ros_head_hokuyo_controller" filename="libgazebo_ros_laser.so">
+                <robotNamespace></robotNamespace>
+                <topicName>laser_scan</topicName>
+                <frameName>hokuyo_laser_link</frameName>
+            </plugin>
+        </sensor>
+    </gazebo>
 </robot>
